Commit message: Training loop with pyo3 + pytorch

File: assets/ant.urdf (robot description, URDF)
Before this commit: robot ant, 9 links, 8 joints
Links:
- removed link front_left_foot
- removed link front_left_leg
- removed link front_right_foot
- removed link front_right_leg
- removed link left_back_foot
- removed link left_back_leg
- removed link right_back_foot
- removed link right_back_leg
- added link back_left_shin, mass 0.1; collision cylinder length=0.3 radius=0.08; visual cylinder length=0.3 radius=0.08
- added link back_left_thigh, mass 0.1; collision cylinder length=0.5 radius=0.08; visual cylinder length=0.5 radius=0.08
- added link back_left_thigh_pitch, mass 0.0
- added link back_right_shin, mass 0.1; collision cylinder length=0.3 radius=0.08; visual cylinder length=0.3 radius=0.08
- added link back_right_thigh, mass 0.1; collision cylinder length=0.5 radius=0.08; visual cylinder length=0.5 radius=0.08
- added link back_right_thigh_pitch, mass 0.0
- added link front_left_shin, mass 0.1; collision cylinder length=0.3 radius=0.08; visual cylinder length=0.3 radius=0.08
- added link front_left_thigh, mass 0.1; collision cylinder length=0.5 radius=0.08; visual cylinder length=0.5 radius=0.08
- added link front_left_thigh_pitch, mass 0.0
- added link front_right_shin, mass 0.1; collision cylinder length=0.3 radius=0.08; visual cylinder length=0.3 radius=0.08
- added link front_right_thigh, mass 0.1; collision cylinder length=0.5 radius=0.08; visual cylinder length=0.5 radius=0.08
- added link front_right_thigh_pitch, mass 0.0
- link torso: mass 1 -> 1.0
Joints:
- removed joint ankle_1
- removed joint ankle_2
- removed joint ankle_3
- removed joint ankle_4
- removed joint hip_1
- removed joint hip_2
- removed joint hip_3
- removed joint hip_4
- added joint hip1_pitch: type revolute, parent front_left_thigh, child front_left_thigh_pitch, origin xyz=0.1 0 -0.08 rpy=0 0 0, axis 0 1 0, limit lower=0 upper=0 effort=100 velocity=1.0
- added joint hip1_roll: type revolute, parent torso, child front_left_thigh, origin xyz=0.2 0.2 0 rpy=0 0 0.7854, axis 0 0 1, limit lower=-0.5 upper=0.5 effort=100 velocity=1.0
- added joint hip2_pitch: type revolute, parent front_right_thigh, child front_right_thigh_pitch, origin xyz=0.1 0 -0.08 rpy=0 0 0, axis 0 1 0, limit lower=0 upper=0 effort=100 velocity=1.0
- added joint hip2_roll: type revolute, parent torso, child front_right_thigh, origin xyz=0.2 -0.2 0 rpy=0 0 -0.7854, axis 0 0 1, limit lower=-0.5 upper=0.5 effort=100 velocity=1.0
- added joint hip3_pitch: type revolute, parent back_left_thigh, child back_left_thigh_pitch, origin xyz=0.1 0 -0.08 rpy=0 0 0, axis 0 1 0, limit lower=0 upper=0 effort=100 velocity=1.0
- added joint hip3_roll: type revolute, parent torso, child back_left_thigh, origin xyz=-0.2 0.2 0 rpy=0 0 2.3562, axis 0 0 1, limit lower=-0.5 upper=0.5 effort=100 velocity=1.0
- added joint hip4_pitch: type revolute, parent back_right_thigh, child back_right_thigh_pitch, origin xyz=0.1 0 -0.08 rpy=0 0 0, axis 0 1 0, limit lower=0 upper=0 effort=100 velocity=1.0
- added joint hip4_roll: type revolute, parent torso, child back_right_thigh, origin xyz=-0.2 -0.2 0 rpy=0 0 -2.3562, axis 0 0 1, limit lower=-0.5 upper=0.5 effort=100 velocity=1.0
- added joint knee1: type revolute, parent front_left_thigh_pitch, child front_left_shin, origin xyz=0.5 0 0 rpy=0 0 0, axis 0 1 0, limit lower=-1.5 upper=0.5 effort=100 velocity=1.0
- added joint knee2: type revolute, parent front_right_thigh_pitch, child front_right_shin, origin xyz=0.5 0 0 rpy=0 0 0, axis 0 1 0, limit lower=-1.5 upper=0.5 effort=100 velocity=1.0
- added joint knee3: type revolute, parent back_left_thigh_pitch, child back_left_shin, origin xyz=0.5 0 0 rpy=0 0 0, axis 0 1 0, limit lower=-1.5 upper=0.5 effort=100 velocity=1.0
- added joint knee4: type revolute, parent back_right_thigh_pitch, child back_right_shin, origin xyz=0.5 0 0 rpy=0 0 0, axis 0 1 0, limit lower=-1.5 upper=0.5 effort=100 velocity=1.0

Commit message: Fixed parameters & model

File: assets/ant.urdf (robot description, URDF)
Before this commit: robot ant, 13 links, 12 joints
Links:
- added link back_left_foot, mass 0.05; collision sphere radius=0.10; visual sphere radius=0.10
- added link back_right_foot, mass 0.05; collision sphere radius=0.10; visual sphere radius=0.10
- added link front_left_foot, mass 0.05; collision sphere radius=0.10; visual sphere radius=0.10
- added link front_right_foot, mass 0.05; collision sphere radius=0.10; visual sphere radius=0.10
Joints:
- added joint back_left_foot_joint: type fixed, parent back_left_shin, child back_left_foot, origin xyz=0 0 -0.45 rpy=0 0 0
- added joint back_right_foot_joint: type fixed, parent back_right_shin, child back_right_foot, origin xyz=0 0 -0.45 rpy=0 0 0
- added joint front_left_foot_joint: type fixed, parent front_left_shin, child front_left_foot, origin xyz=0 0 -0.45 rpy=0 0 0
- added joint front_right_foot_joint: type fixed, parent front_right_shin, child front_right_foot, origin xyz=0 0 -0.45 rpy=0 0 0
